File: V1/eumesmo-rl-4ch12a-nc-v1.kicad_pcb (KiCad board)
At the start: 2 copper layers, 68 x 67.8 mm, 25 parts, among them J1 250-202, J2 250-204, J3 DB142V-5.08-4P, J4 DB142V-5.08-4P, K1 Songle_SRD_1B, K2 Songle_SRD_1B, K3 Songle_SRD_1B, K4 Songle_SRD_1B

Commit message: LEDs changed to orange
Parts:
- D1, D3, D5, D7: value GREEN -> ORANGE/0603
- R1, R2, R3, R4: value 10k/125mW -> 9.1k/125mW
Changed lines of the file:
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@@
 			)
 		)
-		(property "Value" "10k/125mW"
+		(property "Value" "9.1k/125mW"
 			(at 0 1.65 270)
 			(layer "F.Fab")
@@
 			)
 		)
-		(property "Mfr PN" "0805W8F1002T5E"
+		(property "Mfr PN" "0805W8F9101T5E"
 			(at 0 0 270)
 			(unlocked yes)
@@
 			)
 		)
-		(property "Vendor PN" "C17414"
+		(property "Vendor PN" "C17855"
 			(at 0 0 270)
 			(unlocked yes)
@@
 			)
 		)
-		(property "LCSC Part #" "C17414"
+		(property "LCSC Part #" "C17855"
 			(at 0 0 270)
 			(unlocked yes)
@@
 			)
 		)
-		(property "Value" "GREEN"
+		(property "Value" "ORANGE/0603"
 			(at 0 1.43 0)
 			(layer "F.Fab")
@@
 			)
 		)
-		(property "LCSC Part #" "C72043"
+		(property "LCSC Part #" "C2987557"
 			(at 0 0 0)
 			(layer "F.Fab")
@@
 			)
 		)
-		(property "Mfr" "Everlight"
+		(property "Mfr" "Everlight Elec"
 			(at 0 0 0)
 			(layer "F.Fab")
@@
 			)
 		)
-		(property "Mfr PN" "19-217/GHC-YR1S2/3T"
+		(property "Mfr PN" "19-217/S2C-AL1M2VY/6T"
 			(at 0 0 0)
 			(layer "F.Fab")
@@
 			)
 		)
-		(property "Vendor PN" "C72043"
+		(property "Vendor PN" "C2987557"
 			(at 0 0 0)
 			(layer "F.Fab")
@@
 			)
 		)
-		(property "Value" "10k/125mW"
+		(property "Value" "9.1k/125mW"
 			(at 0 1.65 270)
 			(layer "F.Fab")
@@
 			)
 		)
-		(property "Mfr PN" "0805W8F1002T5E"
+		(property "Mfr PN" "0805W8F9101T5E"
 			(at 0 0 270)
 			(unlocked yes)
@@
 			)
 		)
-		(property "Vendor PN" "C17414"
+		(property "Vendor PN" "C17855"
 			(at 0 0 270)
 			(unlocked yes)
@@
 			)
 		)
-		(property "LCSC Part #" "C17414"
+		(property "LCSC Part #" "C17855"
 			(at 0 0 270)
 			(unlocked yes)
@@
 			)
 		)
-		(property "Value" "GREEN"
+		(property "Value" "ORANGE/0603"
 			(at 0 1.43 0)
 			(layer "F.Fab")
@@
 			)
 		)
-		(property "LCSC Part #" "C72043"
+		(property "LCSC Part #" "C2987557"
 			(at 0 0 0)
 			(layer "F.Fab")
@@
 			)
 		)
-		(property "Mfr" "Everlight"
+		(property "Mfr" "Everlight Elec"
 			(at 0 0 0)
 			(layer "F.Fab")
@@
 			)
 		)
-		(property "Mfr PN" "19-217/GHC-YR1S2/3T"
+		(property "Mfr PN" "19-217/S2C-AL1M2VY/6T"
 			(at 0 0 0)
 			(layer "F.Fab")
@@
 			)
 		)
-		(property "Vendor PN" "C72043"
+		(property "Vendor PN" "C2987557"
 			(at 0 0 0)
 			(layer "F.Fab")
@@
 			)
 		)
-		(property "Value" "10k/125mW"
+		(property "Value" "9.1k/125mW"
 			(at 0 1.65 270)
 			(layer "F.Fab")
@@
 			)
 		)
-		(property "Mfr PN" "0805W8F1002T5E"
+		(property "Mfr PN" "0805W8F9101T5E"
 			(at 0 0 270)
 			(unlocked yes)
@@
 			)
 		)
-		(property "Vendor PN" "C17414"
+		(property "Vendor PN" "C17855"
 			(at 0 0 270)
 			(unlocked yes)
@@
 			)
 		)
-		(property "LCSC Part #" "C17414"
+		(property "LCSC Part #" "C17855"
 			(at 0 0 270)
 			(unlocked yes)
@@
 			)
 		)
-		(property "Value" "GREEN"
+		(property "Value" "ORANGE/0603"
 			(at 0 1.43 0)
 			(layer "F.Fab")
@@
 			)
 		)
-		(property "LCSC Part #" "C72043"
+		(property "LCSC Part #" "C2987557"
 			(at 0 0 0)
 			(layer "F.Fab")
@@
 			)
 		)
-		(property "Mfr" "Everlight"
+		(property "Mfr" "Everlight Elec"
 			(at 0 0 0)
 			(layer "F.Fab")
@@
 			)
 		)
-		(property "Mfr PN" "19-217/GHC-YR1S2/3T"
+		(property "Mfr PN" "19-217/S2C-AL1M2VY/6T"
 			(at 0 0 0)
 			(layer "F.Fab")
@@
 			)
 		)
-		(property "Vendor PN" "C72043"
+		(property "Vendor PN" "C2987557"
 			(at 0 0 0)
 			(layer "F.Fab")
@@
 			)
 		)
-		(property "Value" "10k/125mW"
+		(property "Value" "9.1k/125mW"
 			(at 0 1.65 270)
 			(layer "F.Fab")
@@
 			)
 		)
-		(property "Mfr PN" "0805W8F1002T5E"
+		(property "Mfr PN" "0805W8F9101T5E"
 			(at 0 0 270)
 			(unlocked yes)
@@
 			)
 		)
-		(property "Vendor PN" "C17414"
+		(property "Vendor PN" "C17855"
 			(at 0 0 270)
 			(unlocked yes)
@@
 			)
 		)
-		(property "LCSC Part #" "C17414"
+		(property "LCSC Part #" "C17855"
 			(at 0 0 270)
 			(unlocked yes)
@@
 			)
 		)
-		(property "Value" "GREEN"
+		(property "Value" "ORANGE/0603"
 			(at 0 1.43 0)
 			(layer "F.Fab")
@@
 			)
 		)
-		(property "LCSC Part #" "C72043"
+		(property "LCSC Part #" "C2987557"
 			(at 0 0 0)
 			(layer "F.Fab")
@@
 			)
 		)
-		(property "Mfr" "Everlight"
+		(property "Mfr" "Everlight Elec"
 			(at 0 0 0)
 			(layer "F.Fab")
@@
 			)
 		)
-		(property "Mfr PN" "19-217/GHC-YR1S2/3T"
+		(property "Mfr PN" "19-217/S2C-AL1M2VY/6T"
 			(at 0 0 0)
 			(layer "F.Fab")
@@
 			)
 		)
-		(property "Vendor PN" "C72043"
+		(property "Vendor PN" "C2987557"
 			(at 0 0 0)
 			(layer "F.Fab")

Commit message: LEDs replaced for orange
Parts:
- R1, R2, R3, R4: value 9.1k/125mW -> 10k/125mW
Changed lines of the file:
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@@
 			)
 		)
-		(property "Value" "9.1k/125mW"
+		(property "Value" "10k/125mW"
 			(at 0 1.65 270)
 			(layer "F.Fab")
@@
 			)
 		)
-		(property "Mfr PN" "0805W8F9101T5E"
+		(property "Mfr PN" "0805W8F1002T5E"
 			(at 0 0 270)
 			(unlocked yes)
@@
 			)
 		)
-		(property "Vendor PN" "C17855"
+		(property "Vendor PN" "C17414"
 			(at 0 0 270)
 			(unlocked yes)
@@
 			)
 		)
-		(property "LCSC Part #" "C17855"
+		(property "LCSC Part #" "C17414"
 			(at 0 0 270)
 			(unlocked yes)
@@
 			)
 		)
-		(property "Value" "9.1k/125mW"
+		(property "Value" "10k/125mW"
 			(at 0 1.65 270)
 			(layer "F.Fab")
@@
 			)
 		)
-		(property "Mfr PN" "0805W8F9101T5E"
+		(property "Mfr PN" "0805W8F1002T5E"
 			(at 0 0 270)
 			(unlocked yes)
@@
 			)
 		)
-		(property "Vendor PN" "C17855"
+		(property "Vendor PN" "C17414"
 			(at 0 0 270)
 			(unlocked yes)
@@
 			)
 		)
-		(property "LCSC Part #" "C17855"
+		(property "LCSC Part #" "C17414"
 			(at 0 0 270)
 			(unlocked yes)
@@
 			)
 		)
-		(property "Value" "9.1k/125mW"
+		(property "Value" "10k/125mW"
 			(at 0 1.65 270)
 			(layer "F.Fab")
@@
 			)
 		)
-		(property "Mfr PN" "0805W8F9101T5E"
+		(property "Mfr PN" "0805W8F1002T5E"
 			(at 0 0 270)
 			(unlocked yes)
@@
 			)
 		)
-		(property "Vendor PN" "C17855"
+		(property "Vendor PN" "C17414"
 			(at 0 0 270)
 			(unlocked yes)
@@
 			)
 		)
-		(property "LCSC Part #" "C17855"
+		(property "LCSC Part #" "C17414"
 			(at 0 0 270)
 			(unlocked yes)
@@
 			)
 		)
-		(property "Value" "9.1k/125mW"
+		(property "Value" "10k/125mW"
 			(at 0 1.65 270)
 			(layer "F.Fab")
@@
 			)
 		)
-		(property "Mfr PN" "0805W8F9101T5E"
+		(property "Mfr PN" "0805W8F1002T5E"
 			(at 0 0 270)
 			(unlocked yes)
@@
 			)
 		)
-		(property "Vendor PN" "C17855"
+		(property "Vendor PN" "C17414"
 			(at 0 0 270)
 			(unlocked yes)
@@
 			)
 		)
-		(property "LCSC Part #" "C17855"
+		(property "LCSC Part #" "C17414"
 			(at 0 0 270)
 			(unlocked yes)

Commit message: Replaced NC with form C (NO + NC) relays.
Parts:
- added RV5: 275VAC, Tales:RV_Disc_D9.50mm_W3.6mm_P5.08mm, F.Cu at (164.2, 103.2)
- added RV6: 275VAC, Tales:RV_Disc_D9.50mm_W3.6mm_P5.08mm, F.Cu at (169.5, 107.8)
- added RV7: 275VAC, Tales:RV_Disc_D9.50mm_W3.6mm_P5.08mm, F.Cu at (179.5, 103.2)
- added RV8: 275VAC, Tales:RV_Disc_D9.50mm_W3.6mm_P5.08mm, F.Cu at (184.8, 107.8)
- J3, J4: value DB142V-5.08-4P -> DB142V-5.08-6P; footprint Tales:TerminalBlock_Dibo_DB142V-5.08-4P_1x04_P5.08mm_Vertical -> Tales:TerminalBlock_Dibo_DB142V-5.08-6P_1x06_P5.08mm_Vertical
- K1, K2, K3, K4: value Songle_SRD_1B -> Songle_SRD_1C; footprint Tales:Relay_SPST_Songle_SRD_FormB -> Tales:Relay_SPDT_Songle_SRD_FormC
- moved RV4 34.5 mm to (151.2, 108.0)
- moved RV3 23.5 mm to (146.0, 103.5), turned to 180 degrees
- moved RV2 18.1 mm to (136.0, 108.0)
- moved K1 7.16 mm to (133.8, 82.7)
- moved K4 7.16 mm to (184.2, 82.7)
- moved K2 7.07 mm to (150.5, 82.7)
- moved K3 7.07 mm to (167.5, 82.7)
- moved D4 6.82 mm to (150.2, 76.5)
- moved RV1 6.75 mm to (130.8, 103.5), turned to 180 degrees
- moved D2 6.39 mm to (133.8, 76.5)
- moved J3 4.50 mm to (141.0, 118.8)
- moved D6 3.82 mm to (162.2, 76.5)
- moved J4 3.00 mm to (174.5, 118.8)
- moved D8 0.56 mm to (176.5, 79.2)
Connections:
- J3 pad 1: /OUT1PW -> /OUT1NO
- J3 pad 2: /OUT1LD -> /OUT1C
- J3 pad 3: /OUT2PW -> /OUT1NC
- J3 pad 4: /OUT2LD -> /OUT2NO
- J4 pad 1: /OUT3PW -> /OUT3NO
- J4 pad 2: /OUT3LD -> /OUT3C
- J4 pad 3: /OUT4PW -> /OUT3NC
- J4 pad 4: /OUT4LD -> /OUT4NO
- K1 pad 11: /OUT1PW -> /OUT1C
- K1 pad 12: /OUT1LD -> /OUT1NC
- K2 pad 11: /OUT2PW -> /OUT2C
- K2 pad 12: /OUT2LD -> /OUT2NC
- K3 pad 11: /OUT3PW -> /OUT3C
- K3 pad 12: /OUT3LD -> /OUT3NC
- K4 pad 11: /OUT4PW -> /OUT4C
- K4 pad 12: /OUT4LD -> /OUT4NC
- RV1 pad 1: /OUT1PW -> /OUT1C
- RV1 pad 2: /OUT1LD -> /OUT1NO
- RV2 pad 1: /OUT2PW -> /OUT1C
- RV2 pad 2: /OUT2LD -> /OUT1NC
- RV3 pad 1: /OUT3PW -> /OUT2C
- RV3 pad 2: /OUT3LD -> /OUT2NO
- RV4 pad 1: /OUT4PW -> /OUT2C
- RV4 pad 2: /OUT4LD -> /OUT2NC
Routing:
- net /OUT4PW: track 82.3 -> 0.00 mm
- net /OUT2PW: track 82.3 -> 0.00 mm
- net /OUT3PW: track 82.3 -> 0.00 mm
- net /OUT1PW: track 82.3 -> 0.00 mm
- net /OUT4C: track 0.00 -> 81.8 mm
- net /OUT2C: track 0.00 -> 81.6 mm
- net /OUT3C: track 0.00 -> 80.5 mm
- net /OUT1C: track 0.00 -> 80.3 mm
- net /OUT3LD: track 54.6 -> 0.00 mm
- net /OUT1LD: track 54.6 -> 0.00 mm
- net /OUT4LD: track 54.6 -> 0.00 mm
- net /OUT2LD: track 54.6 -> 0.00 mm
- net /OUT4NC: track 0.00 -> 53.8 mm
- net /OUT2NC: track 0.00 -> 53.6 mm
- net /OUT3NC: track 0.00 -> 52.6 mm
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Other:
- outline, holes or cut-outs redrawn
- board text added: "C"
- board text added: "NC"
- board text added: "NO"
- board text added: "eumesmo-rl-4ch12a-c"
- board text removed: "ATTENTION!! NC CONTACTS"
- board text removed: "LOAD"
- board text removed: "V~"
- board text removed: "eumesmo-rl-4ch12a-nc"
