File: V1/eumesmo-rl-4ch12a-c-v1.kicad_sch (KiCad schematic)
At the start: 28 parts, among them J1 250-202, J2 250-204, J3 DB142V-5.08-6P, J4 DB142V-5.08-6P, K1 Songle_SRD_1C, K2 Songle_SRD_1C, K3 Songle_SRD_1C, K4 Songle_SRD_1C

Commit message: Repo renamed.
Other:
- title: eumesmo 4x 24V Relay Module -> eumesmo 4x 24V form C relay Module
Changed lines of the file:
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@@
 	(paper "A4")
 	(title_block
-		(title "eumesmo 4x 24V Relay Module")
-		(date "2026-06-17")
-		(rev "V1.2")
+		(title "eumesmo 4x 24V form C relay Module")
+		(date "2026-09-21")
+		(rev "V1.3")
 	)
 	(text "V_{F} = 1,8V @ 2,5mA\nI_{LED} = (24V - V_{F}) / R\nI_{LED} = (24V - 1.8V) / 10k\nI_{LED} = 2.22 mA"
@@
 		)
 		(instances
-			(project "eumesmo-rl-4ch12a-nc-v1"
+			(project "eumesmo-rl-4ch12a-c-v1"
 				(path "/57cfb5e7-a9ab-4784-80b3-e51e693f5cc8"
 					(reference "#PWR0103")
@@
 		)
 		(instances
-			(project "eumesmo-rl-4ch12a-nc-v1"
+			(project "eumesmo-rl-4ch12a-c-v1"
 				(path "/57cfb5e7-a9ab-4784-80b3-e51e693f5cc8"
 					(reference "D7")
@@
 		)
 		(instances
-			(project "eumesmo-rl-4ch12a-nc-v1"
+			(project "eumesmo-rl-4ch12a-c-v1"
 				(path "/57cfb5e7-a9ab-4784-80b3-e51e693f5cc8"
 					(reference "D2")
@@
 		)
 		(instances
-			(project "eumesmo-rl-4ch12a-nc-v1"
+			(project "eumesmo-rl-4ch12a-c-v1"
 				(path "/57cfb5e7-a9ab-4784-80b3-e51e693f5cc8"
 					(reference "K3")
@@
 		)
 		(instances
-			(project "eumesmo-rl-4ch12a-nc-v1"
+			(project "eumesmo-rl-4ch12a-c-v1"
 				(path "/57cfb5e7-a9ab-4784-80b3-e51e693f5cc8"
 					(reference "J2")
@@
 		)
 		(instances
-			(project "eumesmo-rl-4ch12a-nc-v1"
+			(project "eumesmo-rl-4ch12a-c-v1"
 				(path "/57cfb5e7-a9ab-4784-80b3-e51e693f5cc8"
 					(reference "K2")
@@
 		)
 		(instances
-			(project "eumesmo-rl-4ch12a-nc-v1"
+			(project "eumesmo-rl-4ch12a-c-v1"
 				(path "/57cfb5e7-a9ab-4784-80b3-e51e693f5cc8"
 					(reference "R1")
@@
 		)
 		(instances
-			(project "eumesmo-rl-4ch12a-nc-v1"
+			(project "eumesmo-rl-4ch12a-c-v1"
 				(path "/57cfb5e7-a9ab-4784-80b3-e51e693f5cc8"
 					(reference "#PWR0101")
@@
 		)
 		(instances
-			(project "eumesmo-rl-4ch12a-nc-v1"
+			(project "eumesmo-rl-4ch12a-c-v1"
 				(path "/57cfb5e7-a9ab-4784-80b3-e51e693f5cc8"
 					(reference "#FLG0101")
@@
 		)
 		(instances
-			(project "eumesmo-rl-4ch12a-nc-v1"
+			(project "eumesmo-rl-4ch12a-c-v1"
 				(path "/57cfb5e7-a9ab-4784-80b3-e51e693f5cc8"
 					(reference "D5")
@@
 		)
 		(instances
-			(project "eumesmo-rl-4ch12a-nc-v1"
+			(project "eumesmo-rl-4ch12a-c-v1"
 				(path "/57cfb5e7-a9ab-4784-80b3-e51e693f5cc8"
 					(reference "R3")
@@
 		)
 		(instances
-			(project "eumesmo-rl-4ch12a-nc-v1"
+			(project "eumesmo-rl-4ch12a-c-v1"
 				(path "/57cfb5e7-a9ab-4784-80b3-e51e693f5cc8"
 					(reference "J1")
@@
 		)
 		(instances
-			(project "eumesmo-rl-4ch12a-nc-v1"
+			(project "eumesmo-rl-4ch12a-c-v1"
 				(path "/57cfb5e7-a9ab-4784-80b3-e51e693f5cc8"
 					(reference "J3")
@@
 		)
 		(instances
-			(project "eumesmo-rl-4ch12a-nc-v1"
+			(project "eumesmo-rl-4ch12a-c-v1"
 				(path "/57cfb5e7-a9ab-4784-80b3-e51e693f5cc8"
 					(reference "#PWR0105")
@@
 		)
 		(instances
-			(project "eumesmo-rl-4ch12a-nc-v1"
+			(project "eumesmo-rl-4ch12a-c-v1"
 				(path "/57cfb5e7-a9ab-4784-80b3-e51e693f5cc8"
 					(reference "RV7")
@@
 		)
 		(instances
-			(project "eumesmo-rl-4ch12a-nc-v1"
+			(project "eumesmo-rl-4ch12a-c-v1"
 				(path "/57cfb5e7-a9ab-4784-80b3-e51e693f5cc8"
 					(reference "R4")
@@
 		)
 		(instances
-			(project "eumesmo-rl-4ch12a-nc-v1"
+			(project "eumesmo-rl-4ch12a-c-v1"
 				(path "/57cfb5e7-a9ab-4784-80b3-e51e693f5cc8"
 					(reference "D1")
@@
 		)
 		(instances
-			(project "eumesmo-rl-4ch12a-nc-v1"
+			(project "eumesmo-rl-4ch12a-c-v1"
 				(path "/57cfb5e7-a9ab-4784-80b3-e51e693f5cc8"
 					(reference "RV4")
@@
 		)
 		(instances
-			(project "eumesmo-rl-4ch12a-nc-v1"
+			(project "eumesmo-rl-4ch12a-c-v1"
 				(path "/57cfb5e7-a9ab-4784-80b3-e51e693f5cc8"
 					(reference "RV3")
@@
 		)
 		(instances
-			(project "eumesmo-rl-4ch12a-nc-v1"
+			(project "eumesmo-rl-4ch12a-c-v1"
 				(path "/57cfb5e7-a9ab-4784-80b3-e51e693f5cc8"
 					(reference "J4")
@@
 		)
 		(instances
-			(project "eumesmo-rl-4ch12a-nc-v1"
+			(project "eumesmo-rl-4ch12a-c-v1"
 				(path "/57cfb5e7-a9ab-4784-80b3-e51e693f5cc8"
 					(reference "RV2")
@@
 		)
 		(instances
-			(project "eumesmo-rl-4ch12a-nc-v1"
+			(project "eumesmo-rl-4ch12a-c-v1"
 				(path "/57cfb5e7-a9ab-4784-80b3-e51e693f5cc8"
 					(reference "R2")
@@
 		)
 		(instances
-			(project "eumesmo-rl-4ch12a-nc-v1"
+			(project "eumesmo-rl-4ch12a-c-v1"
 				(path "/57cfb5e7-a9ab-4784-80b3-e51e693f5cc8"
 					(reference "#PWR0104")
@@
 		)
 		(instances
-			(project "eumesmo-rl-4ch12a-nc-v1"
+			(project "eumesmo-rl-4ch12a-c-v1"
 				(path "/57cfb5e7-a9ab-4784-80b3-e51e693f5cc8"
 					(reference "D8")
@@
 		)
 		(instances
-			(project "eumesmo-rl-4ch12a-nc-v1"
+			(project "eumesmo-rl-4ch12a-c-v1"
 				(path "/57cfb5e7-a9ab-4784-80b3-e51e693f5cc8"
 					(reference "#PWR0102")
@@
 		)
 		(instances
-			(project "eumesmo-rl-4ch12a-nc-v1"
+			(project "eumesmo-rl-4ch12a-c-v1"
 				(path "/57cfb5e7-a9ab-4784-80b3-e51e693f5cc8"
 					(reference "RV8")
@@
 		)
 		(instances
-			(project "eumesmo-rl-4ch12a-nc-v1"
+			(project "eumesmo-rl-4ch12a-c-v1"
 				(path "/57cfb5e7-a9ab-4784-80b3-e51e693f5cc8"
 					(reference "D6")
@@
 		)
 		(instances
-			(project "eumesmo-rl-4ch12a-nc-v1"
+			(project "eumesmo-rl-4ch12a-c-v1"
 				(path "/57cfb5e7-a9ab-4784-80b3-e51e693f5cc8"
 					(reference "D3")
@@
 		)
 		(instances
-			(project "eumesmo-rl-4ch12a-nc-v1"
+			(project "eumesmo-rl-4ch12a-c-v1"
 				(path "/57cfb5e7-a9ab-4784-80b3-e51e693f5cc8"
 					(reference "K4")
@@
 		)
 		(instances
-			(project "eumesmo-rl-4ch12a-nc-v1"
+			(project "eumesmo-rl-4ch12a-c-v1"
 				(path "/57cfb5e7-a9ab-4784-80b3-e51e693f5cc8"
 					(reference "D4")
@@
 		)
 		(instances
-			(project "eumesmo-rl-4ch12a-nc-v1"
+			(project "eumesmo-rl-4ch12a-c-v1"
 				(path "/57cfb5e7-a9ab-4784-80b3-e51e693f5cc8"
 					(reference "RV1")
@@
 		)
 		(instances
-			(project "eumesmo-rl-4ch12a-nc-v1"
+			(project "eumesmo-rl-4ch12a-c-v1"
 				(path "/57cfb5e7-a9ab-4784-80b3-e51e693f5cc8"
 					(reference "K1")
@@
 		)
 		(instances
-			(project "eumesmo-rl-4ch12a-nc-v1"
+			(project "eumesmo-rl-4ch12a-c-v1"
 				(path "/57cfb5e7-a9ab-4784-80b3-e51e693f5cc8"
 					(reference "RV6")
@@
 		)
 		(instances
-			(project "eumesmo-rl-4ch12a-nc-v1"
+			(project "eumesmo-rl-4ch12a-c-v1"
 				(path "/57cfb5e7-a9ab-4784-80b3-e51e693f5cc8"
 					(reference "RV5")

Commit message: Updated component visible fields.
Parts:
- RV1, RV2, RV3, RV4, RV5, RV6, RV7, RV8: Technology MOV -> (none)
Changed lines of the file:
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@@
 			)
 		)
-		(property "Technology" "MOV"
+		(property "Technology" ""
 			(at 209.55 132.08 0)
 			(hide yes)
@@
 			)
 		)
-		(property "Technology" "MOV"
+		(property "Technology" ""
 			(at 220.98 62.23 0)
 			(hide yes)
@@
 			)
 		)
-		(property "Technology" "MOV"
+		(property "Technology" ""
 			(at 203.2 62.23 0)
 			(hide yes)
@@
 			)
 		)
-		(property "Technology" "MOV"
+		(property "Technology" ""
 			(at 121.92 62.23 0)
 			(hide yes)
@@
 			)
 		)
-		(property "Technology" "MOV"
+		(property "Technology" ""
 			(at 227.33 132.08 0)
 			(hide yes)
@@
 			)
 		)
-		(property "Technology" "MOV"
+		(property "Technology" ""
 			(at 104.14 54.61 0)
 			(hide yes)
@@
 			)
 		)
-		(property "Technology" "MOV"
+		(property "Technology" ""
 			(at 130.81 132.08 0)
 			(hide yes)
@@
 			)
 		)
-		(property "Technology" "MOV"
+		(property "Technology" ""
 			(at 113.03 124.46 0)
 			(hide yes)

Commit message: Replaced Wago connectors for other brand, no stock.
Parts:
- J1: LCSC Part # C2765061 -> C475154; Mfr Wago -> Cixi Kefa Elec; Mfr PN 250-202 -> KF250-3.5-2P-1; Vendor PN C2765061 -> C475154
- J2: LCSC Part # C2765063 -> C475156; Mfr Wago -> Cixi Kefa Elec; Mfr PN 250-204 -> KF250-3.5-4P-1; Vendor PN C2765063 -> C475156
Changed lines of the file:
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@@
 			)
 		)
-		(property "Mfr" "Wago"
+		(property "Mfr" "Cixi Kefa Elec"
 			(at 27.94 80.01 0)
 			(hide yes)
@@
 			)
 		)
-		(property "LCSC Part #" "C2765063"
+		(property "LCSC Part #" "C475156"
 			(at 27.94 80.01 0)
 			(hide yes)
@@
 			)
 		)
-		(property "Mfr PN" "250-204"
+		(property "Mfr PN" "KF250-3.5-4P-1"
 			(at 27.94 80.01 0)
 			(hide yes)
@@
 			)
 		)
-		(property "Vendor PN" "C2765063"
+		(property "Vendor PN" "C475156"
 			(at 27.94 80.01 0)
 			(hide yes)
@@
 			)
 		)
-		(property "Mfr" "Wago"
+		(property "Mfr" "Cixi Kefa Elec"
 			(at 27.94 181.61 0)
 			(hide yes)
@@
 			)
 		)
-		(property "LCSC Part #" "C2765061"
+		(property "LCSC Part #" "C475154"
 			(at 27.94 181.61 0)
 			(hide yes)
@@
 			)
 		)
-		(property "Mfr PN" "250-202"
+		(property "Mfr PN" "KF250-3.5-2P-1"
 			(at 27.94 181.61 0)
 			(hide yes)
@@
 			)
 		)
-		(property "Vendor PN" "C2765061"
+		(property "Vendor PN" "C475154"
 			(at 27.94 181.61 0)
 			(hide yes)
